Commit message: Update xarm7 urdf: gripper open at q_max

File: mani_skill2/assets/descriptions/xarm7_with_gripper_reduced_dof.urdf (robot description, URDF)
Before this commit: robot xarm7, 14 links, 13 joints
Joints:
- joint left_finger_joint: axis 0 -0.9631963 0.26879897 -> 0 0.9631963 -0.26879897; origin xyz=0 0.07 0.101 rpy=0 0 0 -> xyz=0 0.027 0.113 rpy=0 0 0
- joint right_finger_joint: axis 0. 0.9631963 0.26879897 -> 0. -0.9631963 -0.26879897; origin xyz=0 -0.07 0.101 rpy=0 0 0 -> xyz=0 -0.027 0.113 rpy=0 0 0
