Commit message: Add xarm7_d435 robot urdf

File: mani_skill2/assets/descriptions/xarm7_with_gripper_reduced_dof_d435_v2.urdf (robot description, URDF)
Before this commit: robot xarm7, 14 links, 13 joints
Links:
- added link camera_color_frame
- added link camera_color_optical_frame
- added link camera_depth_frame
- added link camera_depth_optical_frame
- added link camera_left_ir_frame
- added link camera_left_ir_optical_frame
- added link camera_link
- added link camera_right_ir_frame
- added link camera_right_ir_optical_frame
- link link_eef: geometry collision mesh filename=xarm_description/meshes/camera/realsense/collision/d435_wit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; visual mesh filename=xarm_description/meshes/camera/realsense/visual/d435_with_t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
Joints:
- added joint camera_color_joint: type fixed, parent camera_link, child camera_color_frame, origin xyz=0 0.015 0 rpy=0 0 0
- added joint camera_color_optical_joint: type fixed, parent camera_color_frame, child camera_color_optical_frame, origin xyz=0 0 0 rpy=-1.5707963267948966 0 -1.5707963267948966
- added joint camera_depth_joint: type fixed, parent camera_link, child camera_depth_frame, origin xyz=0 0 0 rpy=0 0 0
- added joint camera_depth_optical_joint: type fixed, parent camera_depth_frame, child camera_depth_optical_frame, origin xyz=0 0 0 rpy=-1.5707963267948966 0 -1.5707963267948966
- added joint camera_left_ir_joint: type fixed, parent camera_link, child camera_left_ir_frame, origin xyz=0 0 0 rpy=0 0 0
- added joint camera_left_ir_optical_joint: type fixed, parent camera_left_ir_frame, child camera_left_ir_optical_frame, origin xyz=0 0 0 rpy=-1.5707963267948966 0 -1.5707963267948966
- added joint camera_link_joint: type fixed, parent link_eef, child camera_link, origin xyz=-0.06042734 0.0175 0.02915237 rpy=3.141592653589793 -1.832595714594046 3.141592653589793
- added joint camera_right_ir_joint: type fixed, parent camera_link, child camera_right_ir_frame, origin xyz=0 -0.050 0 rpy=0 0 0
- added joint camera_right_ir_optical_joint: type fixed, parent camera_right_ir_frame, child camera_right_ir_optical_frame, origin xyz=0 0 0 rpy=-1.5707963267948966 0 -1.5707963267948966

Commit message: Fix d435 plate overlapping with gripper_base_link

File: mani_skill2/assets/descriptions/xarm7_with_gripper_reduced_dof_d435_v2.urdf (robot description, URDF)
Before this commit: robot xarm7, 23 links, 22 joints
Joints:
- joint gripper_fix: origin xyz=0 0 0 rpy=0 0 0 -> xyz=0 0 0.005 rpy=0 0 0

File: mani_skill2/assets/descriptions/xarm_floating_textured_reduced_dof_d435_v2.urdf (robot description, URDF)
Before this commit: robot floating_xarm, 21 links, 20 joints
Joints:
- joint gripper_fix: origin xyz=0 0 0 rpy=0 0 0 -> xyz=0 0 0.005 rpy=0 0 0
