Commit message: Add effort to pris joints of floating xarm gripper
* Fix base pose to xarm_gripper_base_link

File: mani_skill2/assets/descriptions/xarm_floating_pris_finger.urdf (robot description, URDF)
Before this commit: robot floating_xarm, 12 links, 11 joints
Joints:
- joint joint_eef: origin xyz=0 0 0 rpy=0 3.141592653589793 0 -> xyz=0 0 0 rpy=0 0 0
- joint x_axis_joint: limit lower=-10 upper=10 velocity=0.50 -> lower=-10 upper=10 effort=50 velocity=0.50
- joint y_axis_joint: limit lower=-10 upper=10 velocity=0.50 -> lower=-10 upper=10 effort=50 velocity=0.50
- joint z_axis_joint: limit lower=-10 upper=10 velocity=0.50 -> lower=-10 upper=10 effort=50 velocity=0.50

File: mani_skill2/assets/descriptions/xarm_floating_pris_finger_d435.urdf (robot description, URDF)
Before this commit: robot floating_xarm, 21 links, 20 joints
Joints:
- joint joint_eef: origin xyz=0 0 0 rpy=0 3.141592653589793 0 -> xyz=0 0 -0.005 rpy=0 0 0
- joint x_axis_joint: limit lower=-10 upper=10 velocity=0.50 -> lower=-10 upper=10 effort=50 velocity=0.50
- joint y_axis_joint: limit lower=-10 upper=10 velocity=0.50 -> lower=-10 upper=10 effort=50 velocity=0.50
- joint z_axis_joint: limit lower=-10 upper=10 velocity=0.50 -> lower=-10 upper=10 effort=50 velocity=0.50
